File: rpi_with_supply/rpi_with_supply.kicad_pcb (KiCad board)
At the start: 2 copper layers, 65 x 56 mm, 48 parts, among them IC1 ATTINY25, J3 Phoenix 1933189 COMBICON, J4 Phoenix 1933189 COMBICON, J5 Raspberry_Pi_2_3, J6 FAN, P1 CONN_1, P10 CONN_02X02, P11 WS2812, P12 UPDI, P2 CONN_1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

Commit message: update design with new switch
Parts:
- C1: value 220uF -> 220uF10v
- C3, C5: value 220uF -> 220uF16v
- R6: value 10k -> 1.5k
- R8: value 1.5k -> 220
- U3: value vn7040-switch -> TPS22810; footprint SOIC-8_3.9x4.9mm_Pitch1.27mm -> SOT-23-6
- moved U3 0.64 mm to (65.6, 67.7), turned to 225 degrees
Connections:
- D6 pad 2: (no net) -> TXRX
- Q2 pad 2: Net-(P12-Pad2) -> HT
- Q2 pad 3: HT -> Net-(P12-Pad2)
- U3 pad 1: INPUT -> +12V
- U3 pad 3: GND -> INPUT
- U3 pad 5: +12V -> (no net)
Routing:
- net OUT: track 27.7 -> 45.8 mm
- net GND: track 482.2 -> 465.1 mm
- net TXRX: track 9.34 -> 13.6 mm, vias 0 -> 2
- net +12V: track 61.8 -> 58.4 mm
- net HT: track 311.7 -> 313.6 mm
Other:
- board text added: "cnpihats rpi_with_supply rev E (C) <>< 2018 C. Lohr"
- board text removed: "cnpihats rpi_with_supply rev D (C) <>< 2018 C. Lohr"
