File: rpi_with_supply/rpi_with_supply.sch (KiCad schematic (older format))
At the start: 50 parts, among them IC1 ATTINY25, J1 Phoenix 1934861, J2 Phoenix 1934861, J3 Phoenix 1933189 COMBICON, J4 Phoenix 1933189 COMBICON, J5 Raspberry_Pi_2_3, J6 FAN, P1 CONN_1, P10 CONN_02X02, P11 WS2812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

Commit message: update design with new switch
Parts:
- removed U3: vn7040-switch, symbol vn7040-switch
- added U3: TPS22810, SOT-23-6, symbol TPS22810-HIGH-SIDE-DRIVER
- C1: value 220uF -> 220uF10v
- C3, C5: value 220uF -> 220uF16v
- R6: value 10k -> 1.5k
- R8: value 1.5k -> 220
Connections:
- net +12V: now also U3.1 (VIN)
- net GND: now also U3.2 (GND)
- net HT: now also Q2.2 (S); no longer Q2.3 (D)
- net INPUT: now also U3.3 (EN)
- net OUT: now also U3.6 (VOUT)
- net TXRX: now also D6.2 (A)
- net at P12.2 (P2), R10.2: now also Q2.3 (D); no longer Q2.2 (S)
Other:
- moved on the sheet: D6
Changed lines of the file:
@@
 LIBS:lm5110
 LIBS:vn7040-switch
+LIBS:tps22810-high-side-driver
 LIBS:rpi_with_supply-cache
 EELAYER 25 0
@@
 P 9200 1100
 F 0 "C3" H 9225 1200 50  0000 L CNN
-F 1 "220uF" H 9225 1000 50  0000 L CNN
+F 1 "220uF16v" H 9225 1000 50  0000 L CNN
 F 2 "CP_Elec_8x6.7" H 9200 1100 50  0001 C CNN
 F 3 "" H 9200 1100 50  0001 C CNN
@@
 P 9900 1100
 F 0 "C5" H 9925 1200 50  0000 L CNN
-F 1 "220uF" H 9925 1000 50  0000 L CNN
+F 1 "220uF16v" H 9925 1000 50  0000 L CNN
 F 2 "CP_Elec_8x6.7" H 9900 1100 50  0001 C CNN
 F 3 "" H 9900 1100 50  0001 C CNN
@@
 P 7150 3350
 F 0 "R6" V 7230 3350 50  0000 C CNN
-F 1 "10k" V 7150 3350 50  0000 C CNN
+F 1 "1.5k" V 7150 3350 50  0000 C CNN
 F 2 "R_0805" V 7080 3350 50  0001 C CNN
 F 3 "" H 7150 3350 50  0001 C CNN
@@
 P 6900 3550
 F 0 "R8" V 6980 3550 50  0000 C CNN
-F 1 "1.5k" V 6900 3550 50  0000 C CNN
+F 1 "220" V 6900 3550 50  0000 C CNN
 F 2 "R_0805" V 6830 3550 50  0001 C CNN
 F 3 "" H 6900 3550 50  0001 C CNN
@@
 P 8500 1100
 F 0 "C1" H 8525 1200 50  0000 L CNN
-F 1 "220uF" H 8525 1000 50  0000 L CNN
+F 1 "220uF10v" H 8525 1000 50  0000 L CNN
 F 2 "CP_Elec_8x6.7" H 8500 1100 50  0001 C CNN
 F 3 "" H 8500 1100 50  0001 C CNN
@@
 L GND #PWR048
 U 1 1 5B2D2CD7
-P 7650 4050
-F 0 "#PWR048" H 7650 3800 50  0001 C CNN
-F 1 "GND" H 7650 3900 50  0000 C CNN
-F 2 "" H 7650 4050 50  0001 C CNN
-F 3 "" H 7650 4050 50  0001 C CNN
-	1    7650 4050
-	0    1    1    0
-$EndComp
-Text GLabel 7650 3850 0    60   Input ~ 0
+P 8000 3300
+F 0 "#PWR048" H 8000 3050 50  0001 C CNN
+F 1 "GND" H 8000 3150 50  0000 C CNN
+F 2 "" H 8000 3300 50  0001 C CNN
+F 3 "" H 8000 3300 50  0001 C CNN
+	1    8000 3300
+	0    1    1    0
+$EndComp
+Text GLabel 8000 3400 0    60   Input ~ 0
 INPUT
 $Comp
-L GND #PWR049
-U 1 1 5B2D2EDB
-P 7650 3950
-F 0 "#PWR049" H 7650 3700 50  0001 C CNN
-F 1 "GND" H 7650 3800 50  0000 C CNN
-F 2 "" H 7650 3950 50  0001 C CNN
-F 3 "" H 7650 3950 50  0001 C CNN
-	1    7650 3950
-	0    1    1    0
-$EndComp
-$Comp
-L +12V #PWR050
-U 1 1 5B2D300C
-P 8650 4150
-F 0 "#PWR050" H 8650 4000 50  0001 C CNN
-F 1 "+12V" H 8650 4290 50  0000 C CNN
-F 2 "" H 8650 4150 50  0001 C CNN
-F 3 "" H 8650 4150 50  0001 C CNN
-	1    8650 4150
-	0    1    1    0
-$EndComp
-$Comp
-L +12V #PWR051
+L +12V #PWR049
 U 1 1 5B2D3083
-P 8650 3850
-F 0 "#PWR051" H 8650 3700 50  0001 C CNN
-F 1 "+12V" H 8650 3990 50  0000 C CNN
-F 2 "" H 8650 3850 50  0001 C CNN
-F 3 "" H 8650 3850 50  0001 C CNN
-	1    8650 3850
-	0    1    1    0
-$EndComp
-Text GLabel 8650 3950 2    60   Input ~ 0
-OUT
-Text GLabel 8650 4050 2    60   Input ~ 0
+P 8000 3200
+F 0 "#PWR049" H 8000 3050 50  0001 C CNN
+F 1 "+12V" H 8000 3340 50  0000 C CNN
+F 2 "" H 8000 3200 50  0001 C CNN
+F 3 "" H 8000 3200 50  0001 C CNN
+	1    8000 3200
+	0    -1   -1   0
+$EndComp
+Text GLabel 8800 3200 2    60   Input ~ 0
 OUT
 Text GLabel 7750 1050 2    60   Input ~ 0
@@
 $EndComp
 $Comp
-L GND #PWR052
+L GND #PWR050
 U 1 1 5B690EB1
 P 4900 7600
-F 0 "#PWR052" H 4900 7350 50  0001 C CNN
+F 0 "#PWR050" H 4900 7350 50  0001 C CNN
 F 1 "GND" H 4900 7450 50  0000 C CNN
 F 2 "" H 4900 7600 50  0001 C CNN
 F 3 "" H 4900 7600 50  0001 C CNN
 	1    4900 7600
-	1    0    0    -1
-$EndComp
-$Comp
-L vn7040-switch U3
-U 1 1 5B78F78C
-P 8150 4000
-F 0 "U3" H 7900 4250 60  0000 C CNN
-F 1 "vn7040-switch" H 8150 3750 60  0000 C CNN
-F 2 "" H 8150 4000 60  0000 C CNN
-F 3 "" H 8150 4000 60  0000 C CNN
-	1    8150 4000
 	1    0    0    -1
 $EndComp
@@
 $EndComp
 $Comp
-L GND #PWR053
+L GND #PWR051
 U 1 1 5B8352B4
 P 5250 6350
-F 0 "#PWR053" H 5250 6100 50  0001 C CNN
+F 0 "#PWR051" H 5250 6100 50  0001 C CNN
 F 1 "GND" H 5250 6200 50  0000 C CNN
 F 2 "" H 5250 6350 50  0001 C CNN
@@
 $EndComp
 $Comp
-L +3.3V #PWR054
+L +3.3V #PWR052
 U 1 1 5B835D56
 P 5250 5850
-F 0 "#PWR054" H 5250 5700 50  0001 C CNN
+F 0 "#PWR052" H 5250 5700 50  0001 C CNN
 F 1 "+3.3V" H 5250 5990 50  0000 C CNN
 F 2 "" H 5250 5850 50  0000 C CNN
@@
 $EndComp
 $Comp
-L +3.3V #PWR055
+L +3.3V #PWR053
 U 1 1 5B838422
 P 5600 6000
-F 0 "#PWR055" H 5600 5850 50  0001 C CNN
+F 0 "#PWR053" H 5600 5850 50  0001 C CNN
 F 1 "+3.3V" H 5600 6140 50  0000 C CNN
 F 2 "" H 5600 6000 50  0000 C CNN
@@
 $EndComp
 $Comp
-L GND #PWR056
+L GND #PWR054
 U 1 1 5B8384A5
 P 5600 6300
-F 0 "#PWR056" H 5600 6050 50  0001 C CNN
+F 0 "#PWR054" H 5600 6050 50  0001 C CNN
 F 1 "GND" H 5600 6150 50  0000 C CNN
 F 2 "" H 5600 6300 50  0001 C CNN
@@
 Connection ~ 2000 6250
 $Comp
-L GND #PWR057
+L GND #PWR055
 U 1 1 5B840229
 P 2000 6600
-F 0 "#PWR057" H 2000 6350 50  0001 C CNN
+F 0 "#PWR055" H 2000 6350 50  0001 C CNN
 F 1 "GND" H 2000 6450 50  0000 C CNN
 F 2 "" H 2000 6600 50  0001 C CNN
@@
 $EndComp
 $Comp
-L HT #PWR058
+L HT #PWR056
 U 1 1 5B8402E0
 P 1950 5950
-F 0 "#PWR058" H 1950 6070 50  0001 C CNN
+F 0 "#PWR056" H 1950 6070 50  0001 C CNN
 F 1 "HT" H 1950 6040 50  0000 C CNN
 F 2 "" H 1950 5950 50  0001 C CNN
@@
 $EndComp
 $Comp
-L GND #PWR059
+L GND #PWR057
 U 1 1 5B8421B7
 P 2900 7350
-F 0 "#PWR059" H 2900 7100 50  0001 C CNN
+F 0 "#PWR057" H 2900 7100 50  0001 C CNN
 F 1 "GND" H 2900 7200 50  0000 C CNN
 F 2 "" H 2900 7350 50  0001 C CNN
@@
 $EndComp
 $Comp
-L GND #PWR060
+L GND #PWR058
 U 1 1 5BC5D089
 P 8900 5550
-F 0 "#PWR060" H 8900 5300 50  0001 C CNN
+F 0 "#PWR058" H 8900 5300 50  0001 C CNN
 F 1 "GND" H 8900 5400 50  0000 C CNN
 F 2 "" H 8900 5550 50  0001 C CNN
@@
 $EndComp
 $Comp
-L GND #PWR061
+L GND #PWR059
 U 1 1 5BD4A366
 P 4450 3200
-F 0 "#PWR061" H 4450 2950 50  0001 C CNN
+F 0 "#PWR059" H 4450 2950 50  0001 C CNN
 F 1 "GND" H 4450 3050 50  0000 C CNN
 F 2 "" H 4450 3200 50  0001 C CNN
@@
 L LED-RESCUE-rpi_with_supply D6
 U 1 1 5BD4B84C
-P 4350 3800
-F 0 "D6" H 4350 3900 50  0000 C CNN
-F 1 "BLU" H 4350 3700 50  0000 C CNN
-F 2 "LED_0805" H 4350 3800 50  0001 C CNN
-F 3 "" H 4350 3800 50  0001 C CNN
-	1    4350 3800
+P 4350 3850
+F 0 "D6" H 4350 3950 50  0000 C CNN
+F 1 "BLU" H 4350 3750 50  0000 C CNN
+F 2 "LED_0805" H 4350 3850 50  0001 C CNN
+F 3 "" H 4350 3850 50  0001 C CNN
+	1    4350 3850
 	0    1    -1   0
 $EndComp
 $Comp
-L GND #PWR062
+L GND #PWR060
 U 1 1 5BD4CB7A
-P 4350 3950
-F 0 "#PWR062" H 4350 3700 50  0001 C CNN
-F 1 "GND" H 4350 3800 50  0000 C CNN
-F 2 "" H 4350 3950 50  0001 C CNN
-F 3 "" H 4350 3950 50  0001 C CNN
-	1    4350 3950
-	0    1    1    0
-$EndComp
-$Comp
-L +3.3V #PWR063
+P 4350 4000
+F 0 "#PWR060" H 4350 3750 50  0001 C CNN
+F 1 "GND" H 4350 3850 50  0000 C CNN
+F 2 "" H 4350 4000 50  0001 C CNN
+F 3 "" H 4350 4000 50  0001 C CNN
+	1    4350 4000
+	0    1    1    0
+$EndComp
+$Comp
+L +3.3V #PWR061
 U 1 1 5BD4FD64
 P 4450 3000
-F 0 "#PWR063" H 4450 2850 50  0001 C CNN
+F 0 "#PWR061" H 4450 2850 50  0001 C CNN
 F 1 "+3.3V" H 4450 3140 50  0000 C CNN
 F 2 "" H 4450 3000 50  0000 C CNN
@@
 $EndComp
 $Comp
-L +3.3V #PWR064
+L +3.3V #PWR062
 U 1 1 5BD4FE2B
 P 2700 1650
-F 0 "#PWR064" H 2700 1500 50  0001 C CNN
+F 0 "#PWR062" H 2700 1500 50  0001 C CNN
 F 1 "+3.3V" H 2700 1790 50  0000 C CNN
 F 2 "" H 2700 1650 50  0000 C CNN
@@
 $EndComp
 $Comp
-L HT #PWR065
+L HT #PWR063
 U 1 1 5BD52EB6
 P 4950 2150
-F 0 "#PWR065" H 4950 2270 50  0001 C CNN
+F 0 "#PWR063" H 4950 2270 50  0001 C CNN
 F 1 "HT" H 4950 2240 50  0000 C CNN
 F 2 "" H 4950 2150 50  0001 C CNN
@@
 $EndComp
 $Comp
-L HT #PWR066
+L HT #PWR064
 U 1 1 5BD53A26
 P 4150 1850
-F 0 "#PWR066" H 4150 1970 50  0001 C CNN
+F 0 "#PWR064" H 4150 1970 50  0001 C CNN
 F 1 "HT" H 4150 1940 50  0000 C CNN
 F 2 "" H 4150 1850 50  0001 C CNN
@@
 	4200 3100 4450 3100
 $Comp
-L GND #PWR067
+L GND #PWR065
 U 1 1 5BD57BD3
 P 4150 2650
-F 0 "#PWR067" H 4150 2400 50  0001 C CNN
+F 0 "#PWR065" H 4150 2400 50  0001 C CNN
 F 1 "GND" H 4150 2500 50  0000 C CNN
 F 2 "" H 4150 2650 50  0001 C CNN
@@
 F 4 "FDV304PCT-ND‎" H 4850 2350 60  0001 C CNN "Digikey"
 	1    4850 2350
-	1    0    0    -1
+	1    0    0    1
 $EndComp
 Wire Wire Line
@@
 	4950 2750 4200 2750
 Connection ~ 4200 3100
+Text GLabel 4350 3700 0    60   Input ~ 0
+TXRX
+$Comp
+L TPS22810-HIGH-SIDE-DRIVER U3
+U 1 1 5BDCD7DB
+P 8400 3300
+F 0 "U3" H 8250 3500 60  0000 C CNN
+F 1 "TPS22810" H 8400 3100 60  0000 C CNN
+F 2 "SOT-23-6" H 8400 3300 60  0000 C CNN
+F 3 "" H 8400 3300 60  0000 C CNN
+	1    8400 3300
+	1    0    0    -1
+$EndComp
 $EndSCHEMATC
