File: rpi_esp_flasher/rpi_esp_flasher.kicad_pcb (KiCad board)
At the start: 2 copper layers, 31 x 32.5 mm, 19 parts, among them J1 Raspberry_Pi_2_3, P1 ESP, P4 CONN_1, SW1 PWR, U1 4427, U2 1117_5v_or_3v, U3 1k

Commit message: switch to LM5110
Parts:
- U1: value 4427 -> LM5110
Connections:
- U1 pad 1: (no net) -> GND
- U1 pad 2: (no net) -> GPIO2
- U1 pad 7: (no net) -> Net-(D6-Pad2)
Routing:
- net GND: track 116.4 -> 110.4 mm
- net GPIO2: track 11.6 -> 16.3 mm
- net Net-(D6-Pad2): track 23.5 -> 27.8 mm
Other:
- board text added: "cnpihats rpi_esp_flasher rev A (C) <>< 2018 C. Lohr"
- board text removed: "cnpihats rpi_esp_flasher rev - (C) <>< 2018 C. Lohr"
Changed lines of the file:
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@@
 (kicad_pcb (version 4) (host pcbnew 4.0.2+dfsg1-stable)
   (general
-    (links 39)
+    (links 42)
     (no_connects 0)
     (area 14.224 14.732 87.884001 73.152001)
     (thickness 1.6)
     (drawings 21)
-    (tracks 224)
+    (tracks 230)
     (zones 0)
     (modules 19)
@@
       (drillshape 0)
       (scaleselection 1)
-      (outputdirectory rpi_esp_flasher_rev-))
+      (outputdirectory rpi_esp_flasher_revA))
   )
   (net 0 "")
@@
       (effects (font (size 1 1) (thickness 0.15)))
     )
-    (fp_text value 4427 (at 4.5 0 180) (layer F.SilkS)
+    (fp_text value LM5110 (at 4.4 -0.81 180) (layer F.SilkS)
       (effects (font (size 1 1) (thickness 0.15)))
     )
@@
     (fp_line (start -2.075 2.575) (end 2.075 2.575) (layer F.SilkS) (width 0.15))
     (fp_line (start -2.075 -2.43) (end -3.475 -2.43) (layer F.SilkS) (width 0.15))
-    (pad 1 smd rect (at -2.7 -1.905 90) (size 1.55 0.6) (layers F.Cu F.Paste F.Mask))
-    (pad 2 smd rect (at -2.7 -0.635 90) (size 1.55 0.6) (layers F.Cu F.Paste F.Mask))
+    (pad 1 smd rect (at -2.7 -1.905 90) (size 1.55 0.6) (layers F.Cu F.Paste F.Mask)
+      (net 2 GND))
+    (pad 2 smd rect (at -2.7 -0.635 90) (size 1.55 0.6) (layers F.Cu F.Paste F.Mask)
+      (net 14 GPIO2))
     (pad 3 smd rect (at -2.7 0.635 90) (size 1.55 0.6) (layers F.Cu F.Paste F.Mask)
       (net 2 GND))
@@
     (pad 6 smd rect (at 2.7 0.635 90) (size 1.55 0.6) (layers F.Cu F.Paste F.Mask)
       (net 3 "Net-(C7-Pad2)"))
-    (pad 7 smd rect (at 2.7 -0.635 90) (size 1.55 0.6) (layers F.Cu F.Paste F.Mask))
+    (pad 7 smd rect (at 2.7 -0.635 90) (size 1.55 0.6) (layers F.Cu F.Paste F.Mask)
+      (net 12 "Net-(D6-Pad2)"))
     (pad 8 smd rect (at 2.7 -1.905 90) (size 1.55 0.6) (layers F.Cu F.Paste F.Mask))
     (model Housings_SOIC.3dshapes/SOIC-8_3.9x4.9mm_Pitch1.27mm.wrl
@@
   (gr_line (start 35.5 60.5) (end 63 60.5) (angle 90) (layer Edge.Cuts) (width 0.15))
   (gr_arc (start 35.5 57) (end 35.5 60.5) (angle 90) (layer Edge.Cuts) (width 0.15))
-  (gr_text "cnpihats\nrpi_esp_flasher rev -\n(C) <>< 2018 C. Lohr" (at 47.625 48.895) (layer B.SilkS)
+  (gr_text "cnpihats\nrpi_esp_flasher rev A\n(C) <>< 2018 C. Lohr" (at 47.625 48.895) (layer B.SilkS)
     (effects (font (size 1.5 1.5) (thickness 0.3)) (justify mirror))
   )
@@
   (via (at 42.83 46.42) (size 0.6) (drill 0.4) (layers F.Cu B.Cu) (net 2))
   (segment (start 42.415 46.835) (end 42.83 46.42) (width 0.3302) (layer F.Cu) (net 2))
-  (segment (start 41.2 40.43) (end 42.22 40.43) (width 0.3302) (layer F.Cu) (net 2) (status 400000))
+  (segment (start 41.2 40.43) (end 42.22 40.43) (width 0.3302) (layer F.Cu) (net 2))
   (segment (start 42.46 40.65) (end 42.47 40.65) (width 0.3302) (layer B.Cu) (net 2))
   (segment (start 42.45 40.66) (end 42.46 40.65) (width 0.3302) (layer B.Cu) (net 2))
@@
   (segment (start 44.34 29.44) (end 44.34 31.05) (width 0.3302) (layer B.Cu) (net 2))
   (segment (start 44.37 29.41) (end 44.34 29.44) (width 0.3302) (layer B.Cu) (net 2))
-  (segment (start 38 30) (end 38.08 30) (width 0.3302) (layer B.Cu) (net 2) (status C00000))
-  (segment (start 38.08 30) (end 39.54 28.54) (width 0.3302) (layer B.Cu) (net 2) (status 400000))
+  (segment (start 38 30) (end 38.08 30) (width 0.3302) (layer B.Cu) (net 2))
+  (segment (start 38.08 30) (end 39.54 28.54) (width 0.3302) (layer B.Cu) (net 2))
   (segment (start 46.91 29.12) (end 46.91 30.63) (width 0.3302) (layer B.Cu) (net 2))
   (segment (start 46.33 28.54) (end 46.91 29.12) (width 0.3302) (layer B.Cu) (net 2))
@@
   (segment (start 44.34 29.14) (end 44.34 30.548224) (width 0.3302) (layer F.Cu) (net 2))
   (segment (start 43.68 28.48) (end 44.34 29.14) (width 0.3302) (layer F.Cu) (net 2))
-  (segment (start 38 30) (end 38.06 30) (width 0.3302) (layer F.Cu) (net 2) (status C00000))
-  (segment (start 38.06 30) (end 39.58 28.48) (width 0.3302) (layer F.Cu) (net 2) (status 400000))
+  (segment (start 38 30) (end 38.06 30) (width 0.3302) (layer F.Cu) (net 2))
+  (segment (start 38.06 30) (end 39.58 28.48) (width 0.3302) (layer F.Cu) (net 2))
   (segment (start 41.81 29.01) (end 41.81 31.05) (width 0.3302) (layer F.Cu) (net 2))
   (segment (start 41.28 28.48) (end 41.81 29.01) (width 0.3302) (layer F.Cu) (net 2))
@@
   (segment (start 42.335 46.835) (end 41 45.5) (width 0.3302) (layer F.Cu) (net 2))
   (segment (start 41 45.5) (end 40.86 45.5) (width 0.3302) (layer F.Cu) (net 2))
-  (segment (start 40.86 45.5) (end 39.37 46.99) (width 0.3302) (layer F.Cu) (net 2))
-  (segment (start 39.37 46.99) (end 37.465 46.99) (width 0.3302) (layer F.Cu) (net 2))
-  (segment (start 37.465 46.99) (end 36.635 47.82) (width 0.3302) (layer F.Cu) (net 2))
-  (segment (start 36.635 47.82) (end 36.635 48.7) (width 0.3302) (layer F.Cu) (net 2))
   (segment (start 46 43.698) (end 46 42.81) (width 0.27) (layer F.Cu) (net 3))
   (segment (start 46 42.81) (end 47.3 41.51) (width 0.27) (layer F.Cu) (net 3))
@@
   (segment (start 60 35.54902) (end 60 38.05) (width 0.27) (layer F.Cu) (net 5))
   (segment (start 60 38.05) (end 59 39.05) (width 0.27) (layer F.Cu) (net 5))
-  (segment (start 45 33.45098) (end 44.49098 33.45098) (width 0.27) (layer F.Cu) (net 6) (status C00000))
-  (segment (start 44.49098 33.45098) (end 43.08 32.04) (width 0.27) (layer F.Cu) (net 6) (status 400000))
-  (segment (start 43.08 32.04) (end 43.08 30) (width 0.27) (layer F.Cu) (net 6) (status 800000))
+  (segment (start 45 33.45098) (end 44.49098 33.45098) (width 0.27) (layer F.Cu) (net 6))
+  (segment (start 44.49098 33.45098) (end 43.08 32.04) (width 0.27) (layer F.Cu) (net 6))
+  (segment (start 43.08 32.04) (end 43.08 30) (width 0.27) (layer F.Cu) (net 6))
   (segment (start 45 39.05) (end 44.46 39.05) (width 0.27) (layer F.Cu) (net 6))
   (segment (start 44.46 39.05) (end 43.63 38.22) (width 0.27) (layer F.Cu) (net 6))
@@
   (segment (start 51.65 37.17) (end 42.04 37.17) (width 0.27) (layer F.Cu) (net 11))
   (segment (start 53.27098 35.54902) (end 51.65 37.17) (width 0.27) (layer F.Cu) (net 11))
+  (segment (start 35.365 43.3) (end 35.365 42.745) (width 0.27) (layer F.Cu) (net 12) (status C00000))
+  (segment (start 35.365 42.745) (end 36 42.11) (width 0.27) (layer F.Cu) (net 12) (status 400000))
+  (segment (start 36 42.11) (end 37.49 42.11) (width 0.27) (layer F.Cu) (net 12))
+  (segment (start 37.49 42.11) (end 37.905 42.525) (width 0.27) (layer F.Cu) (net 12) (status 800000))
+  (segment (start 37.905 42.525) (end 37.905 43.3) (width 0.27) (layer F.Cu) (net 12) (status C00000))
   (segment (start 37.905 43.3) (end 37.905 42.325) (width 0.27) (layer F.Cu) (net 12))
   (segment (start 47.36 35.05) (end 47.36 32.09) (width 0.27) (layer F.Cu) (net 12))
@@
   (segment (start 51.39 35.81) (end 51.12902 35.54902) (width 0.27) (layer F.Cu) (net 13))
   (segment (start 51.12902 35.54902) (end 50 35.54902) (width 0.27) (layer F.Cu) (net 13))
+  (segment (start 37.905 48.7) (end 37.905 47.955) (width 0.27) (layer F.Cu) (net 14) (status C00000))
+  (segment (start 37.905 47.955) (end 37.32 47.37) (width 0.27) (layer F.Cu) (net 14) (status 400000))
+  (segment (start 35.365 47.785) (end 35.365 48.7) (width 0.27) (layer F.Cu) (net 14) (status 800000))
+  (segment (start 35.78 47.37) (end 35.365 47.785) (width 0.27) (layer F.Cu) (net 14))
+  (segment (start 37.32 47.37) (end 35.78 47.37) (width 0.27) (layer F.Cu) (net 14))
   (segment (start 42.91 58.27) (end 42.91 57.92) (width 0.27) (layer B.Cu) (net 14))
   (segment (start 42.91 57.92) (end 41.65 56.66) (width 0.27) (layer B.Cu) (net 14))

Commit message: Update revb with new switch
Parts:
- U1: value LM5110 -> TPS22810; footprint SOIC-8_3.9x4.9mm_Pitch1.27mm -> SOT-23-6
- moved C7 4.77 mm to (39.5, 49.0), turned to 180 degrees
- moved U1 4.26 mm to (40.3, 45.9)
Connections:
- U1 pad 1: GND -> Net-(C7-Pad2)
- U1 pad 2: GPIO2 -> GND
- U1 pad 3: GND -> GPIO2
- U1 pad 4: GPIO2 -> (no net)
- U1 pad 5: Net-(D6-Pad2) -> (no net)
- U1 pad 6: Net-(C7-Pad2) -> Net-(D6-Pad2)
Routing:
- net Net-(D6-Pad2): track 27.8 -> 24.8 mm
- net GPIO2: track 16.3 -> 13.4 mm
- net GND: track 110.4 -> 113.1 mm, vias 4 -> 6
Other:
- board text added: "cnpihats rpi_esp_flasher rev B (C) <>< 2018 C. Lohr"
- board text removed: "cnpihats rpi_esp_flasher rev A (C) <>< 2018 C. Lohr"
